File: hardware/Device-on-bag/Device-on-bag.kicad_pcb (KiCad board)
At the start: 2 copper layers, 51.4 x 37.2 mm, 4 parts, among them J1 Conn_01x12, J2 Conn_01x12

Commit message: update
Parts:
- removed the REF** at (142.3, 84.1)
- removed the REF** at (119.4, 84.1)
- added REF**: PinSocket_1x10_P2.54mm_Vertical, Connector_PinSocket_2.54mm:PinSocket_1x10_P2.54mm_Vertical, F.Cu at (91.3, 55.2)
- added REF**: PinSocket_1x10_P2.54mm_Vertical, Connector_PinSocket_2.54mm:PinSocket_1x10_P2.54mm_Vertical, F.Cu at (114.2, 55.3)
- moved J1 40.2 mm to (136.9, 81.0)
- moved J2 40.2 mm to (121.7, 81.0)
Connections:
- J1 pad 1: 3v3 -> (no net)
- J1 pad 10: unconnected-(J1-Pad10) -> (no net)
- J1 pad 11: unconnected-(J1-Pad11) -> (no net)
- J1 pad 2: unconnected-(J1-Pad2) -> (no net)
- J1 pad 3: unconnected-(J1-Pad3) -> (no net)
- J1 pad 4: unconnected-(J1-Pad4) -> (no net)
- J1 pad 5: unconnected-(J1-Pad5) -> (no net)
- J1 pad 6: unconnected-(J1-Pad6) -> (no net)
- J1 pad 7: unconnected-(J1-Pad7) -> (no net)
- J1 pad 8: unconnected-(J1-Pad8) -> (no net)
- J1 pad 9: unconnected-(J1-Pad9) -> (no net)
- J2 pad 1: GND -> (no net)
- J2 pad 10: unconnected-(J2-Pad10) -> (no net)
- J2 pad 11: unconnected-(J2-Pad11) -> (no net)
- J2 pad 2: unconnected-(J2-Pad2) -> (no net)
- J2 pad 3: unconnected-(J2-Pad3) -> (no net)
- J2 pad 4: unconnected-(J2-Pad4) -> (no net)
- J2 pad 5: unconnected-(J2-Pad5) -> (no net)
- J2 pad 6: unconnected-(J2-Pad6) -> (no net)
- J2 pad 7: unconnected-(J2-Pad7) -> (no net)
- J2 pad 8: SCL -> (no net)
- J2 pad 9: SDA -> (no net)
Routing:
- net (no net): track 0.00 -> 121.2 mm
- net 3v3: track 52.2 -> 0.00 mm
- net SDA: track 35.7 -> 0.00 mm
- net GND: track 24.7 -> 0.00 mm
- net SCL: track 8.67 -> 0.00 mm

Commit message: update
Parts:
- removed J1, J2: Conn_01x12, Connector_PinSocket_2.54mm:PinSocket_1x11_P2.54mm_Vertical
- removed REF** (x2): PinSocket_1x10_P2.54mm_Vertical, Connector_PinSocket_2.54mm:PinSocket_1x10_P2.54mm_Vertical
- added U1: SparkFun_SEN-14480_H3LIS331DL, SparkFun_Tri_Axis_Accel_Breakout-H3LIS331DL:SparkFun_Tri_Axis_Accel_Breakout-H3LIS331DL, F.Cu at (182.9, 83.8)
- added U2: ESP32-DEVKIT-V1, ESP32-DEVKIT-V1:MODULE_ESP32_DEVKIT_V1, F.Cu at (156.7, 99.1)
Routing:
- net (no net): track 121.2 -> 0.00 mm
Other:
- board size 51.4 x 37.2 mm -> 58.4 x 58.4 mm

Commit message: update
Parts:
- added J1: Conn_01x08, Connector_PinSocket_2.54mm:PinSocket_1x08_P2.54mm_Vertical, F.Cu at (63.4, 86.4)
- added J2: Conn_01x08, Connector_PinSocket_2.54mm:PinSocket_1x08_P2.54mm_Vertical, F.Cu at (63.4, 63.5)
- moved U1 133.8 mm to (54.6, 45.7)
- moved U2 82.3 mm to (83.8, 61.0)
Connections:
- U2 pad 11: unconnected-(U2-Pad11) -> SDA
- U2 pad 14: unconnected-(U2-Pad14) -> SCL
- U2 pad 2: unconnected-(U2-Pad2) -> GND
- U2 pad 21: SDA -> unconnected-(U2-Pad21)
- U2 pad 22: SCL -> unconnected-(U2-Pad22)
- U2 pad 29: GND -> unconnected-(U2-Pad29)
- U2 pad 30: unconnected-(U2-Pad30) -> Vin
Routing:
- net 3.3V: track 0.00 -> 103.4 mm
- net SDA: track 0.00 -> 94.7 mm
- net SCL: track 0.00 -> 74.8 mm
- net Vin: track 0.00 -> 29.0 mm
- net GND: track 0.00 -> 2.46 mm
- added copper zone on F.Cu, net GND
Other:
- board size 58.4 x 58.4 mm -> 66 x 64.1 mm

Commit message: update
Parts:
- removed the J1 at (63.4, 86.4)
- removed the J2 at (63.4, 63.5)
- removed U1: SparkFun_SEN-14480_H3LIS331DL, SparkFun_Tri_Axis_Accel_Breakout-H3LIS331DL:SparkFun_Tri_Axis_Accel_Breakout-H3LIS331DL
- removed the U2 at (83.8, 61.0)
- added J1: Conn_01x08, Connector_PinSocket_2.54mm:PinSocket_1x08_P2.54mm_Vertical, F.Cu at (74.3, 181.5)
- added J1: Conn_01x08, Connector_PinSocket_2.54mm:PinSocket_1x08_P2.54mm_Vertical, F.Cu at (219.1, 180.4)
- added J1: Conn_01x08, Connector_PinSocket_2.54mm:PinSocket_1x08_P2.54mm_Vertical, F.Cu at (219.1, 77.1)
- added J1: Conn_01x08, Connector_PinSocket_2.54mm:PinSocket_1x08_P2.54mm_Vertical, F.Cu at (74.3, 78.3)
- added J2: Conn_01x08, Connector_PinSocket_2.54mm:PinSocket_1x08_P2.54mm_Vertical, F.Cu at (74.3, 57.9)
- added J2: Conn_01x08, Connector_PinSocket_2.54mm:PinSocket_1x08_P2.54mm_Vertical, F.Cu at (219.1, 160.0)
- added J2: Conn_01x08, Connector_PinSocket_2.54mm:PinSocket_1x08_P2.54mm_Vertical, F.Cu at (219.1, 56.8)
- added J2: Conn_01x08, Connector_PinSocket_2.54mm:PinSocket_1x08_P2.54mm_Vertical, F.Cu at (74.3, 161.2)
- added J3: Conn_01x12, Connector_PinSocket_2.54mm:PinSocket_1x12_P2.54mm_Vertical, F.Cu at (191.2, 49.1)
- added J3: Conn_01x12, Connector_PinSocket_2.54mm:PinSocket_1x12_P2.54mm_Vertical, F.Cu at (46.4, 50.2)
- added J3: Conn_01x12, Connector_PinSocket_2.54mm:PinSocket_1x12_P2.54mm_Vertical, F.Cu at (46.4, 153.5)
- added J3: Conn_01x12, Connector_PinSocket_2.54mm:PinSocket_1x12_P2.54mm_Vertical, F.Cu at (191.2, 152.3)
- added J4: Conn_01x12, Connector_PinSocket_2.54mm:PinSocket_1x12_P2.54mm_Vertical, F.Cu at (219.1, 137.2)
- added J4: Conn_01x12, Connector_PinSocket_2.54mm:PinSocket_1x12_P2.54mm_Vertical, F.Cu at (74.3, 35.1)
- added J4: Conn_01x12, Connector_PinSocket_2.54mm:PinSocket_1x12_P2.54mm_Vertical, F.Cu at (74.3, 138.3)
- added J4: Conn_01x12, Connector_PinSocket_2.54mm:PinSocket_1x12_P2.54mm_Vertical, F.Cu at (219.1, 33.9)
- added U2: ESP32-DEVKIT-V1, ESP32-DEVKIT-V1:MODULE_ESP32_DEVKIT_V1, F.Cu at (94.0, 57.3)
- added U2: ESP32-DEVKIT-V1, ESP32-DEVKIT-V1:MODULE_ESP32_DEVKIT_V1, F.Cu at (238.8, 159.4)
- added U2: ESP32-DEVKIT-V1, ESP32-DEVKIT-V1:MODULE_ESP32_DEVKIT_V1, F.Cu at (94.0, 160.5)
- added U2: ESP32-DEVKIT-V1, ESP32-DEVKIT-V1:MODULE_ESP32_DEVKIT_V1, F.Cu at (238.8, 56.2)
Routing:
- net Vin: track 29.0 -> 335.8 mm
- net SCL: track 74.8 -> 311.0 mm
- net SDA: track 94.7 -> 255.7 mm
- net GND: track 2.46 -> 77.5 mm
- net 3.3V: track 103.4 -> 157.9 mm
Other:
- board size 66 x 64.1 mm -> 213.4 x 160.2 mm

Commit message: hardware update
Parts:
- removed the J1 at (74.3, 181.5)
- removed the J1 at (219.1, 180.4)
- removed the J1 at (219.1, 77.1)
- removed the J2 at (219.1, 160.0)
- removed the J2 at (219.1, 56.8)
- removed the J2 at (74.3, 161.2)
- removed the J3 at (191.2, 49.1)
- removed the J3 at (46.4, 153.5)
- removed the J3 at (191.2, 152.3)
- removed the J4 at (219.1, 137.2)
- removed the J4 at (74.3, 138.3)
- removed the J4 at (219.1, 33.9)
- removed the U2 at (238.8, 159.4)
- removed the U2 at (94.0, 160.5)
- removed the U2 at (238.8, 56.2)
- moved J4 5.16 mm to (74.3, 29.9)
- moved J3 5.16 mm to (46.4, 45.1)
- moved J2 2.67 mm to (74.3, 55.3)
- moved J1 0.16 mm to (74.3, 78.1)
Routing:
- net Vin: track 335.8 -> 83.4 mm
- net SCL: track 311.0 -> 75.5 mm
- net SDA: track 255.7 -> 66.3 mm
- net 3.3V: track 157.9 -> 36.6 mm
- net GND: track 77.5 -> 17.4 mm
Other:
- board size 213.4 x 160.2 mm -> 68.6 x 59.1 mm

Commit message: update hardware
Parts:
- moved J1 4.45 mm to (74.3, 73.7)
- moved J2 4.45 mm to (74.3, 50.8)
- moved U2 3.94 mm to (94.0, 53.3)
Connections:
- J4 pad 10: unconnected-(J4-Pad10) -> 3.3V
Routing:
- net GND: track 17.4 -> 4.80 mm
- net 3.3V: track 36.6 -> 48.2 mm
- net Vin: track 83.4 -> 94.8 mm
- net SCL: track 75.5 -> 71.8 mm
- net SDA: track 66.3 -> 63.4 mm
Other:
- board size 68.6 x 59.1 mm -> 67.3 x 56.5 mm

Commit message: update
Parts:
- removed J3, J4: Conn_01x12, Connector_PinSocket_2.54mm:PinSocket_1x12_P2.54mm_Vertical
- added U1: STEVAL-MKI215V1, STEVAL-MKI215V1:STEVAL-MKI215V1, F.Cu at (60.3, 36.8)
