File: hardware/Device-on-bag/Device-on-bag.kicad_sch (KiCad schematic)
At the start: 5 parts, among them J1 Conn_01x08, J2 Conn_01x08, J3 Conn_01x12, J4 Conn_01x12, U2 ESP32-DEVKIT-V1

Commit message: update
Parts:
- removed J3, J4: Conn_01x12, Connector_PinSocket_2.54mm:PinSocket_1x12_P2.54mm_Vertical, symbol Connector_Generic:Conn_01x12
- added U1: STEVAL-MKI215V1, STEVAL-MKI215V1:STEVAL-MKI215V1, symbol STEVAL-MKI215V1:STEVAL-MKI215V1
Connections:
- net 3.3V: now also U1.1 (VDD), U1.22 (SDO)
- net SCL: now also U1.20 (SCL)
- net SDA: now also U1.21 (SDA)
Changed lines of the file:
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@@
 (kicad_sch (version 20211123) (generator eeschema)
   (paper "A4")
-  (global_label "SDA" (shape input) (at 91.44 92.71 0) (fields_autoplaced)
-    (effects (font (size 1.27 1.27)) (justify left))
-    (property "Intersheet References" "${INTERSHEET_REFS}" (id 0) (at 97.4212 92.6306 0)
-      (effects (font (size 1.27 1.27)) (justify left) hide)
-    )
-  )
   (global_label "GND" (shape input) (at 193.04 119.38 0) (fields_autoplaced)
     (effects (font (size 1.27 1.27)) (justify left))
     (property "Intersheet References" "${INTERSHEET_REFS}" (id 0) (at 199.3236 119.4594 0)
-      (effects (font (size 1.27 1.27)) (justify left) hide)
-    )
-  )
-  (global_label "3.3V" (shape input) (at 91.44 90.17 0) (fields_autoplaced)
-    (effects (font (size 1.27 1.27)) (justify left))
-    (property "Intersheet References" "${INTERSHEET_REFS}" (id 0) (at 97.9655 90.0906 0)
       (effects (font (size 1.27 1.27)) (justify left) hide)
     )
@@
     )
   )
-  (global_label "GND" (shape input) (at 91.44 113.03 0) (fields_autoplaced)
-    (effects (font (size 1.27 1.27)) (justify left))
-    (property "Intersheet References" "${INTERSHEET_REFS}" (id 0) (at 97.7236 113.1094 0)
-      (effects (font (size 1.27 1.27)) (justify left) hide)
+  (global_label "SCL" (shape input) (at 123.825 53.975 180) (fields_autoplaced)
+    (effects (font (size 1.27 1.27)) (justify right))
+    (property "Intersheet References" "${INTERSHEET_REFS}" (id 0) (at 117.9043 54.0544 0)
+      (effects (font (size 1.27 1.27)) (justify right) hide)
+    )
+  )
+  (global_label "3.3V" (shape input) (at 123.825 61.595 180) (fields_autoplaced)
+    (effects (font (size 1.27 1.27)) (justify right))
+    (property "Intersheet References" "${INTERSHEET_REFS}" (id 0) (at 117.2995 61.6744 0)
+      (effects (font (size 1.27 1.27)) (justify right) hide)
     )
   )
@@
     )
   )
+  (global_label "3.3V" (shape input) (at 140.335 60.325 0) (fields_autoplaced)
+    (effects (font (size 1.27 1.27)) (justify left))
+    (property "Intersheet References" "${INTERSHEET_REFS}" (id 0) (at 146.8605 60.2456 0)
+      (effects (font (size 1.27 1.27)) (justify left) hide)
+    )
+  )
   (global_label "3.3V" (shape input) (at 193.04 73.66 0) (fields_autoplaced)
     (effects (font (size 1.27 1.27)) (justify left))
     (property "Intersheet References" "${INTERSHEET_REFS}" (id 0) (at 199.5655 73.5806 0)
       (effects (font (size 1.27 1.27)) (justify left) hide)
-    )
-  )
-  (global_label "3.3V" (shape input) (at 73.025 85.09 180) (fields_autoplaced)
-    (effects (font (size 1.27 1.27)) (justify right))
-    (property "Intersheet References" "${INTERSHEET_REFS}" (id 0) (at 66.4995 85.1694 0)
-      (effects (font (size 1.27 1.27)) (justify right) hide)
     )
   )
@@
     )
   )
-  (global_label "SCL" (shape input) (at 91.44 95.25 0) (fields_autoplaced)
-    (effects (font (size 1.27 1.27)) (justify left))
-    (property "Intersheet References" "${INTERSHEET_REFS}" (id 0) (at 97.3607 95.1706 0)
-      (effects (font (size 1.27 1.27)) (justify left) hide)
-    )
-  )
   (global_label "SCL" (shape input) (at 193.04 96.52 0) (fields_autoplaced)
     (effects (font (size 1.27 1.27)) (justify left))
     (property "Intersheet References" "${INTERSHEET_REFS}" (id 0) (at 198.9607 96.4406 0)
       (effects (font (size 1.27 1.27)) (justify left) hide)
+    )
+  )
+  (global_label "SDA" (shape input) (at 123.825 57.785 180) (fields_autoplaced)
+    (effects (font (size 1.27 1.27)) (justify right))
+    (property "Intersheet References" "${INTERSHEET_REFS}" (id 0) (at 117.8438 57.8644 0)
+      (effects (font (size 1.27 1.27)) (justify right) hide)
     )
   )
@@
     (pin "7")
     (pin "8")
-  )
-  (symbol (lib_id "Connector_Generic:Conn_01x12") (at 78.105 97.79 0) (unit 1)
-    (in_bom yes) (on_board yes) (fields_autoplaced)
-    (property "Reference" "J3" (id 0) (at 81.28 97.7899 0)
-      (effects (font (size 1.27 1.27)) (justify left))
-    )
-    (property "Value" "Conn_01x12" (id 1) (at 81.28 100.3299 0)
-      (effects (font (size 1.27 1.27)) (justify left))
-    )
-    (property "Footprint" "Connector_PinSocket_2.54mm:PinSocket_1x12_P2.54mm_Vertical" (id 2) (at 78.105 97.79 0)
-      (effects (font (size 1.27 1.27)) hide)
-    )
-    (property "Datasheet" "~" (id 3) (at 78.105 97.79 0)
-      (effects (font (size 1.27 1.27)) hide)
-    )
-    (pin "1")
-    (pin "10")
-    (pin "11")
-    (pin "12")
-    (pin "2")
-    (pin "3")
-    (pin "4")
-    (pin "5")
-    (pin "6")
-    (pin "7")
-    (pin "8")
-    (pin "9")
   )
   (symbol (lib_id "Connector_Generic:Conn_01x08") (at 114.3 134.62 0) (unit 1)
@@
     (pin "8")
   )
-  (symbol (lib_id "Connector_Generic:Conn_01x12") (at 86.36 100.33 180) (unit 1)
+  (symbol (lib_id "STEVAL-MKI215V1:STEVAL-MKI215V1") (at 132.08 57.15 0) (unit 1)
     (in_bom yes) (on_board yes) (fields_autoplaced)
-    (property "Reference" "J4" (id 0) (at 86.36 78.105 0))
-    (property "Value" "Conn_01x12" (id 1) (at 86.36 80.645 0))
-    (property "Footprint" "Connector_PinSocket_2.54mm:PinSocket_1x12_P2.54mm_Vertical" (id 2) (at 86.36 100.33 0)
+    (property "Reference" "U1" (id 0) (at 132.08 45.72 0))
+    (property "Value" "STEVAL-MKI215V1" (id 1) (at 132.08 48.26 0))
+    (property "Footprint" "STEVAL-MKI215V1:STEVAL-MKI215V1" (id 2) (at 118.745 53.975 0)
       (effects (font (size 1.27 1.27)) hide)
     )
-    (property "Datasheet" "~" (id 3) (at 86.36 100.33 0)
+    (property "Datasheet" "" (id 3) (at 118.745 53.975 0)
       (effects (font (size 1.27 1.27)) hide)
     )
     (pin "1")
-    (pin "10")
-    (pin "11")
-    (pin "12")
-    (pin "2")
-    (pin "3")
-    (pin "4")
-    (pin "5")
-    (pin "6")
-    (pin "7")
-    (pin "8")
-    (pin "9")
+    (pin "13")
+    (pin "20")
+    (pin "21")
+    (pin "22")
   )
   (symbol (lib_id "ESP32-DEVKIT-V1:ESP32-DEVKIT-V1") (at 177.8 99.06 0) (unit 1)
@@
       (reference "J2") (unit 1) (value "Conn_01x08") (footprint "Connector_PinSocket_2.54mm:PinSocket_1x08_P2.54mm_Vertical")
     )
-    (path "/752f9595-3eb9-4010-a3c3-154e60e73472"
-      (reference "J3") (unit 1) (value "Conn_01x12") (footprint "Connector_PinSocket_2.54mm:PinSocket_1x12_P2.54mm_Vertical")
-    )
-    (path "/ec14a061-dfd4-4b23-b005-a6397276b0b5"
-      (reference "J4") (unit 1) (value "Conn_01x12") (footprint "Connector_PinSocket_2.54mm:PinSocket_1x12_P2.54mm_Vertical")
+    (path "/9fa4e663-d7d4-4000-a762-eea9f272de72"
+      (reference "U1") (unit 1) (value "STEVAL-MKI215V1") (footprint "STEVAL-MKI215V1:STEVAL-MKI215V1")
     )
     (path "/f3434164-7b41-4e11-b256-2613206fdd17"
