File: hardware/Device-on-bag/Device-on-bag.kicad_sch (KiCad schematic)
At the start: 5 parts, among them J1 Conn_01x08, J2 Conn_01x08, J3 Conn_01x12, J4 Conn_01x12, U2 ESP32-DEVKIT-V1

Commit message: update
Parts:
- removed J3, J4: Conn_01x12, Connector_PinSocket_2.54mm:PinSocket_1x12_P2.54mm_Vertical, symbol Connector_Generic:Conn_01x12
- added U1: STEVAL-MKI215V1, STEVAL-MKI215V1:STEVAL-MKI215V1, symbol STEVAL-MKI215V1:STEVAL-MKI215V1
Connections:
- net 3.3V: now also U1.1 (VDD), U1.22 (SDO)
- net GND: now also U1.13 (GND)
- net SCL: now also U1.20 (SCL)
- net SDA: now also U1.21 (SDA)
Changed lines of the file:
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@@
 (kicad_sch (version 20211123) (generator eeschema)
   (paper "A4")
-  (global_label "SDA" (shape input) (at 91.44 92.71 0) (fields_autoplaced)
-    (effects (font (size 1.27 1.27)) (justify left))
-    (property "Intersheet References" "${INTERSHEET_REFS}" (id 0) (at 97.4212 92.6306 0)
-      (effects (font (size 1.27 1.27)) (justify left) hide)
-    )
-  )
   (global_label "GND" (shape input) (at 193.04 119.38 0) (fields_autoplaced)
     (effects (font (size 1.27 1.27)) (justify left))
@@
     )
   )
-  (global_label "3.3V" (shape input) (at 91.44 90.17 0) (fields_autoplaced)
-    (effects (font (size 1.27 1.27)) (justify left))
-    (property "Intersheet References" "${INTERSHEET_REFS}" (id 0) (at 97.9655 90.0906 0)
-      (effects (font (size 1.27 1.27)) (justify left) hide)
-    )
-  )
   (global_label "Vin" (shape input) (at 109.22 144.78 180) (fields_autoplaced)
     (effects (font (size 1.27 1.27)) (justify right))
@@
     )
   )
+  (global_label "3.3V" (shape input) (at 139.065 81.28 0) (fields_autoplaced)
+    (effects (font (size 1.27 1.27)) (justify left))
+    (property "Intersheet References" "${INTERSHEET_REFS}" (id 0) (at 145.5905 81.2006 0)
+      (effects (font (size 1.27 1.27)) (justify left) hide)
+    )
+  )
+  (global_label "3.3V" (shape input) (at 122.555 82.55 180) (fields_autoplaced)
+    (effects (font (size 1.27 1.27)) (justify right))
+    (property "Intersheet References" "${INTERSHEET_REFS}" (id 0) (at 116.0295 82.6294 0)
+      (effects (font (size 1.27 1.27)) (justify right) hide)
+    )
+  )
   (global_label "Vin" (shape input) (at 162.56 73.66 180) (fields_autoplaced)
     (effects (font (size 1.27 1.27)) (justify right))
@@
     )
   )
-  (global_label "GND" (shape input) (at 91.44 113.03 0) (fields_autoplaced)
-    (effects (font (size 1.27 1.27)) (justify left))
-    (property "Intersheet References" "${INTERSHEET_REFS}" (id 0) (at 97.7236 113.1094 0)
-      (effects (font (size 1.27 1.27)) (justify left) hide)
-    )
-  )
   (global_label "GND" (shape input) (at 193.04 121.92 0) (fields_autoplaced)
     (effects (font (size 1.27 1.27)) (justify left))
@@
     )
   )
+  (global_label "GND" (shape input) (at 139.065 76.2 0) (fields_autoplaced)
+    (effects (font (size 1.27 1.27)) (justify left))
+    (property "Intersheet References" "${INTERSHEET_REFS}" (id 0) (at 145.3486 76.2794 0)
+      (effects (font (size 1.27 1.27)) (justify left) hide)
+    )
+  )
+  (global_label "SCL" (shape input) (at 122.555 74.93 180) (fields_autoplaced)
+    (effects (font (size 1.27 1.27)) (justify right))
+    (property "Intersheet References" "${INTERSHEET_REFS}" (id 0) (at 116.6343 75.0094 0)
+      (effects (font (size 1.27 1.27)) (justify right) hide)
+    )
+  )
   (global_label "3.3V" (shape input) (at 193.04 73.66 0) (fields_autoplaced)
     (effects (font (size 1.27 1.27)) (justify left))
@@
     )
   )
-  (global_label "3.3V" (shape input) (at 73.025 85.09 180) (fields_autoplaced)
-    (effects (font (size 1.27 1.27)) (justify right))
-    (property "Intersheet References" "${INTERSHEET_REFS}" (id 0) (at 66.4995 85.1694 0)
-      (effects (font (size 1.27 1.27)) (justify right) hide)
-    )
-  )
   (global_label "SDA" (shape input) (at 162.56 119.38 180) (fields_autoplaced)
     (effects (font (size 1.27 1.27)) (justify right))
@@
     )
   )
-  (global_label "SCL" (shape input) (at 91.44 95.25 0) (fields_autoplaced)
-    (effects (font (size 1.27 1.27)) (justify left))
-    (property "Intersheet References" "${INTERSHEET_REFS}" (id 0) (at 97.3607 95.1706 0)
-      (effects (font (size 1.27 1.27)) (justify left) hide)
+  (global_label "SDA" (shape input) (at 122.555 78.74 180) (fields_autoplaced)
+    (effects (font (size 1.27 1.27)) (justify right))
+    (property "Intersheet References" "${INTERSHEET_REFS}" (id 0) (at 116.5738 78.8194 0)
+      (effects (font (size 1.27 1.27)) (justify right) hide)
     )
   )
@@
     (pin "8")
   )
-  (symbol (lib_id "Connector_Generic:Conn_01x12") (at 78.105 97.79 0) (unit 1)
-    (in_bom yes) (on_board yes) (fields_autoplaced)
-    (property "Reference" "J3" (id 0) (at 81.28 97.7899 0)
+  (symbol (lib_id "STEVAL-MKI215V1:STEVAL-MKI215V1") (at 130.81 78.105 0) (unit 1)
+    (in_bom yes) (on_board yes) (fields_autoplaced)
+    (property "Reference" "U1" (id 0) (at 130.81 66.04 0))
+    (property "Value" "STEVAL-MKI215V1" (id 1) (at 130.81 68.58 0))
+    (property "Footprint" "STEVAL-MKI215V1:STEVAL-MKI215V1" (id 2) (at 117.475 74.93 0)
+      (effects (font (size 1.27 1.27)) hide)
+    )
+    (property "Datasheet" "" (id 3) (at 117.475 74.93 0)
+      (effects (font (size 1.27 1.27)) hide)
+    )
+    (pin "1")
+    (pin "13")
+    (pin "20")
+    (pin "21")
+    (pin "22")
+  )
+  (symbol (lib_id "Connector_Generic:Conn_01x08") (at 114.3 134.62 0) (unit 1)
+    (in_bom yes) (on_board yes) (fields_autoplaced)
+    (property "Reference" "J1" (id 0) (at 116.84 134.6199 0)
       (effects (font (size 1.27 1.27)) (justify left))
     )
-    (property "Value" "Conn_01x12" (id 1) (at 81.28 100.3299 0)
+    (property "Value" "Conn_01x08" (id 1) (at 116.84 137.1599 0)
       (effects (font (size 1.27 1.27)) (justify left))
     )
-    (property "Footprint" "Connector_PinSocket_2.54mm:PinSocket_1x12_P2.54mm_Vertical" (id 2) (at 78.105 97.79 0)
-      (effects (font (size 1.27 1.27)) hide)
-    )
-    (property "Datasheet" "~" (id 3) (at 78.105 97.79 0)
-      (effects (font (size 1.27 1.27)) hide)
-    )
-    (pin "1")
-    (pin "10")
-    (pin "11")
-    (pin "12")
+    (property "Footprint" "Connector_PinSocket_2.54mm:PinSocket_1x08_P2.54mm_Vertical" (id 2) (at 114.3 134.62 0)
+      (effects (font (size 1.27 1.27)) hide)
+    )
+    (property "Datasheet" "~" (id 3) (at 114.3 134.62 0)
+      (effects (font (size 1.27 1.27)) hide)
+    )
+    (pin "1")
     (pin "2")
     (pin "3")
@@
     (pin "7")
     (pin "8")
-    (pin "9")
-  )
-  (symbol (lib_id "Connector_Generic:Conn_01x08") (at 114.3 134.62 0) (unit 1)
-    (in_bom yes) (on_board yes) (fields_autoplaced)
-    (property "Reference" "J1" (id 0) (at 116.84 134.6199 0)
-      (effects (font (size 1.27 1.27)) (justify left))
-    )
-    (property "Value" "Conn_01x08" (id 1) (at 116.84 137.1599 0)
-      (effects (font (size 1.27 1.27)) (justify left))
-    )
-    (property "Footprint" "Connector_PinSocket_2.54mm:PinSocket_1x08_P2.54mm_Vertical" (id 2) (at 114.3 134.62 0)
-      (effects (font (size 1.27 1.27)) hide)
-    )
-    (property "Datasheet" "~" (id 3) (at 114.3 134.62 0)
-      (effects (font (size 1.27 1.27)) hide)
-    )
-    (pin "1")
-    (pin "2")
-    (pin "3")
-    (pin "4")
-    (pin "5")
-    (pin "6")
-    (pin "7")
-    (pin "8")
-  )
-  (symbol (lib_id "Connector_Generic:Conn_01x12") (at 86.36 100.33 180) (unit 1)
-    (in_bom yes) (on_board yes) (fields_autoplaced)
-    (property "Reference" "J4" (id 0) (at 86.36 78.105 0))
-    (property "Value" "Conn_01x12" (id 1) (at 86.36 80.645 0))
-    (property "Footprint" "Connector_PinSocket_2.54mm:PinSocket_1x12_P2.54mm_Vertical" (id 2) (at 86.36 100.33 0)
-      (effects (font (size 1.27 1.27)) hide)
-    )
-    (property "Datasheet" "~" (id 3) (at 86.36 100.33 0)
-      (effects (font (size 1.27 1.27)) hide)
-    )
-    (pin "1")
-    (pin "10")
-    (pin "11")
-    (pin "12")
-    (pin "2")
-    (pin "3")
-    (pin "4")
-    (pin "5")
-    (pin "6")
-    (pin "7")
-    (pin "8")
-    (pin "9")
   )
   (symbol (lib_id "ESP32-DEVKIT-V1:ESP32-DEVKIT-V1") (at 177.8 99.06 0) (unit 1)
@@
       (reference "J2") (unit 1) (value "Conn_01x08") (footprint "Connector_PinSocket_2.54mm:PinSocket_1x08_P2.54mm_Vertical")
     )
-    (path "/752f9595-3eb9-4010-a3c3-154e60e73472"
-      (reference "J3") (unit 1) (value "Conn_01x12") (footprint "Connector_PinSocket_2.54mm:PinSocket_1x12_P2.54mm_Vertical")
-    )
-    (path "/ec14a061-dfd4-4b23-b005-a6397276b0b5"
-      (reference "J4") (unit 1) (value "Conn_01x12") (footprint "Connector_PinSocket_2.54mm:PinSocket_1x12_P2.54mm_Vertical")
+    (path "/2c448bb6-b5e9-495b-8c7f-7bcce18622d6"
+      (reference "U1") (unit 1) (value "STEVAL-MKI215V1") (footprint "STEVAL-MKI215V1:STEVAL-MKI215V1")
     )
     (path "/f3434164-7b41-4e11-b256-2613206fdd17"

Commit message: update device on bag hardware
Parts:
- removed J1, J2: Conn_01x08, Connector_PinSocket_2.54mm:PinSocket_1x08_P2.54mm_Vertical, symbol Connector_Generic:Conn_01x08
- added U3: D1_mini_battery_shield, D1 mini battery shield:D1 mini battery shield, symbol d1 mini battery shield:D1_mini_battery_shield
Connections:
- net GND: now also U3.10 (GND)
- net Vin: now also U3.9 (5V)
Changed lines of the file:
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@@
     )
   )
-  (global_label "Vin" (shape input) (at 109.22 144.78 180) (fields_autoplaced)
+  (global_label "Vin" (shape input) (at 103.505 92.71 180) (fields_autoplaced)
     (effects (font (size 1.27 1.27)) (justify right))
-    (property "Intersheet References" "${INTERSHEET_REFS}" (id 0) (at 103.9645 144.7006 0)
+    (property "Intersheet References" "${INTERSHEET_REFS}" (id 0) (at 98.2495 92.6306 0)
       (effects (font (size 1.27 1.27)) (justify right) hide)
     )
@@
     )
   )
-  (global_label "GND" (shape input) (at 109.22 142.24 180) (fields_autoplaced)
-    (effects (font (size 1.27 1.27)) (justify right))
-    (property "Intersheet References" "${INTERSHEET_REFS}" (id 0) (at 102.9364 142.1606 0)
-      (effects (font (size 1.27 1.27)) (justify right) hide)
-    )
-  )
   (global_label "GND" (shape input) (at 139.065 76.2 0) (fields_autoplaced)
     (effects (font (size 1.27 1.27)) (justify left))
     (property "Intersheet References" "${INTERSHEET_REFS}" (id 0) (at 145.3486 76.2794 0)
       (effects (font (size 1.27 1.27)) (justify left) hide)
+    )
+  )
+  (global_label "GND" (shape input) (at 103.505 95.885 180) (fields_autoplaced)
+    (effects (font (size 1.27 1.27)) (justify right))
+    (property "Intersheet References" "${INTERSHEET_REFS}" (id 0) (at 97.2214 95.8056 0)
+      (effects (font (size 1.27 1.27)) (justify right) hide)
     )
   )
@@
     )
   )
-  (symbol (lib_id "Connector_Generic:Conn_01x08") (at 119.38 137.16 180) (unit 1)
-    (in_bom yes) (on_board yes) (fields_autoplaced)
-    (property "Reference" "J2" (id 0) (at 119.38 120.65 0))
-    (property "Value" "Conn_01x08" (id 1) (at 119.38 123.19 0))
-    (property "Footprint" "Connector_PinSocket_2.54mm:PinSocket_1x08_P2.54mm_Vertical" (id 2) (at 119.38 137.16 0)
-      (effects (font (size 1.27 1.27)) hide)
-    )
-    (property "Datasheet" "~" (id 3) (at 119.38 137.16 0)
-      (effects (font (size 1.27 1.27)) hide)
-    )
-    (pin "1")
-    (pin "2")
-    (pin "3")
-    (pin "4")
-    (pin "5")
-    (pin "6")
-    (pin "7")
-    (pin "8")
-  )
   (symbol (lib_id "STEVAL-MKI215V1:STEVAL-MKI215V1") (at 130.81 78.105 0) (unit 1)
     (in_bom yes) (on_board yes) (fields_autoplaced)
@@
     (pin "22")
   )
-  (symbol (lib_id "Connector_Generic:Conn_01x08") (at 114.3 134.62 0) (unit 1)
+  (symbol (lib_id "d1 mini battery shield:D1_mini_battery_shield") (at 107.315 97.79 0) (unit 1)
     (in_bom yes) (on_board yes) (fields_autoplaced)
-    (property "Reference" "J1" (id 0) (at 116.84 134.6199 0)
+    (property "Reference" "U3" (id 0) (at 113.03 93.0274 0)
       (effects (font (size 1.27 1.27)) (justify left))
     )
-    (property "Value" "Conn_01x08" (id 1) (at 116.84 137.1599 0)
+    (property "Value" "D1_mini_battery_shield" (id 1) (at 113.03 95.5674 0)
       (effects (font (size 1.27 1.27)) (justify left))
     )
-    (property "Footprint" "Connector_PinSocket_2.54mm:PinSocket_1x08_P2.54mm_Vertical" (id 2) (at 114.3 134.62 0)
+    (property "Footprint" "D1 mini battery shield:D1 mini battery shield" (id 2) (at 107.315 97.79 0)
       (effects (font (size 1.27 1.27)) hide)
     )
-    (property "Datasheet" "~" (id 3) (at 114.3 134.62 0)
+    (property "Datasheet" "" (id 3) (at 107.315 97.79 0)
       (effects (font (size 1.27 1.27)) hide)
     )
-    (pin "1")
-    (pin "2")
-    (pin "3")
-    (pin "4")
-    (pin "5")
-    (pin "6")
-    (pin "7")
-    (pin "8")
+    (pin "10")
+    (pin "9")
   )
   (symbol (lib_id "ESP32-DEVKIT-V1:ESP32-DEVKIT-V1") (at 177.8 99.06 0) (unit 1)
@@
   )
   (symbol_instances
-    (path "/8e909e36-2ea6-4b97-ad8a-8a0879639875"
-      (reference "J1") (unit 1) (value "Conn_01x08") (footprint "Connector_PinSocket_2.54mm:PinSocket_1x08_P2.54mm_Vertical")
-    )
-    (path "/173b3a26-c401-4096-bbdf-e51853bf08d7"
-      (reference "J2") (unit 1) (value "Conn_01x08") (footprint "Connector_PinSocket_2.54mm:PinSocket_1x08_P2.54mm_Vertical")
-    )
     (path "/2c448bb6-b5e9-495b-8c7f-7bcce18622d6"
       (reference "U1") (unit 1) (value "STEVAL-MKI215V1") (footprint "STEVAL-MKI215V1:STEVAL-MKI215V1")
@@
       (reference "U2") (unit 1) (value "ESP32-DEVKIT-V1") (footprint "MODULE_ESP32_DEVKIT_V1")
     )
+    (path "/74ec461f-c738-4af4-8051-1d9d12808726"
+      (reference "U3") (unit 1) (value "D1_mini_battery_shield") (footprint "D1 mini battery shield:D1 mini battery shield")
+    )
   )
