File: hardware/loacell/loacell.kicad_pcb (KiCad board)
At the start: 2 copper layers, 7 parts, among them J1 Conn_01x04_Male, U1 INA128, U2 D1_mini_battery_shield, U3 ESP32-DEVKIT-V1

Commit message: init
Parts:
- moved U3 144.8 mm to (33.0, 41.0)
- moved U1 125.9 mm to (52.2, 19.2)
- moved J1 111.0 mm to (75.0, 19.2)
- moved JP1 103.6 mm to (54.0, 44.5)
- moved RV1 100.0 mm to (56.5, 61.0), turned to 0 degrees
- moved R1 97.4 mm to (59.0, 34.0), turned to 180 degrees
- moved U2 94.0 mm to (72.0, 45.9), turned to 0 degrees
Routing:
- net GND: track 0.00 -> 85.4 mm
- net lc_input+: track 0.00 -> 59.1 mm
- net Net-(U2-5V): track 0.00 -> 50.4 mm
- net Net-(R1-Pad1): track 0.00 -> 45.7 mm
- net lc_amp_output: track 0.00 -> 44.1 mm
- net Net-(JP1-C): track 0.00 -> 30.9 mm
- net lc_output+: track 0.00 -> 28.6 mm
- net lc_output-: track 0.00 -> 23.9 mm
- net Net-(JP1-B): track 0.00 -> 12.5 mm
- net Net-(JP1-A): track 0.00 -> 11.5 mm
- added copper zone on B.Cu, net GND
- added copper zone on F.Cu, net GND
Other:
- board outline added: 70 x 50 mm
